File: AoE_Too_Hot.kicad_sch (KiCad schematic)
At the start: 8 parts, among them U1 LMV393

Commit message: Add files via upload
Parts:
- removed U1: LMV393, Package_DIP:DIP-8_W7.62mm_LongPads, symbol Comparator:LMV393
- added U1: MCP6562, Package_DIP:DIP-8_W7.62mm_LongPads, symbol Comparator:MCP6562
- BT1: footprint Battery:BatteryHolder_Keystone_2460_1xAA -> Battery:BatteryHolder_Multicomp_BC-2001_1x2032
- D1: footprint Diode_THT:D_A-405_P10.16mm_Horizontal -> LED_THT:LED_D3.0mm_IRBlack
- renumbered R5 to R4
Connections:
- net GND: now also U1.4 (V-)
- net at BT1.1 (+), D1.2 (A), R1.1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: now also U1.8 (V+)
- net at R1.2, R2.1: now also U1.3 (+)
- net at R4.2: now also U1.1
- net at R3.2, TH1.1: now also U1.2 (-)
