File: AoE_Too_Hot.kicad_sch (KiCad schematic)
At the start: 8 parts, among them U1 MCP6562

Commit message: Add files via upload
Parts:
- removed U1: MCP6562, Package_DIP:DIP-8_W7.62mm_LongPads, symbol Comparator:MCP6562
- added U1: LM393, Package_DIP:DIP-8_W7.62mm_LongPads, symbol Comparator:LM393
- BT1: footprint Battery:BatteryHolder_Multicomp_BC-2001_1x2032 -> Battery:BatteryHolder_MPD_BC2003_1x2032
- D1: footprint LED_THT:LED_D3.0mm_IRBlack -> LED_THT:LED_D3.0mm
Connections:
- net GND: now also U1.4 (V-)
- net at BT1.1 (+), D1.2 (A), R1.1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: now also U1.8 (V+)
- net at R1.2, R2.1: now also U1.3 (+)
- net at R4.2: now also U1.1
- net at R3.2, TH1.1: now also U1.2 (-)
